Commit message: add launcher

File: golem_description/urdf/golem_simple.urdf (robot description, URDF)
Before this commit: robot golem, 3 links, 2 joints
Links:
- link base_link: geometry collision mesh filename=package://golem_description/models/golembase.dae; visual mesh filename=package://golem_description/models/golembase.dae
- link wheel_l1: geometry collision mesh filename=package://golem_description/models/llanta2.dae; visual mesh filename=package://golem_description/models/llanta2.dae
- link wheel_r1: geometry collision mesh filename=package://golem_description/models/llanta2.dae; visual mesh filename=package://golem_description/models/llanta2.dae
